File: ODRIVE_V1.0.kicad_pcb (KiCad board)
At the start: 2 copper layers, 167.3 x 165 mm, 48 parts, among them J1 USB_B, J10 RJ11-6N-B, J11 Screw_Terminal_01x02, J12 Screw_Terminal_01x02, J3 Screw_Terminal_01x02, J4 Conn_01x02_Pin, J5 Conn_01x08_Pin, J6 Conn_01x08_Pin, J8 Conn_01x04_Pin, SW3 SW_DPST_x2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

Commit message: updating to finals
Parts:
- removed C19, C20: 22UF, Capacitor_THT:CP_Radial_D8.0mm_P3.50mm
- added C23: 22UF, Capacitor_THT:CP_Radial_D5.0mm_P2.50mm, F.Cu at (54.4, 164.1)
- added C24: 22UF, Capacitor_THT:CP_Radial_D5.0mm_P2.50mm, F.Cu at (61.2, 155.7)
- added D2: 1N4148, Diode_THT:D_DO-35_SOD27_P7.62mm_Horizontal, F.Cu at (35.1, 145.3)
- added D3: 1N4148, Diode_THT:D_DO-35_SOD27_P7.62mm_Horizontal, F.Cu at (35.1, 141.3)
- added J2: Screw_Terminal_01x02, TerminalBlock:TerminalBlock_Altech_AK300-2_P5.00mm, F.Cu at (17.7, 31.1)
- added J7: USB4110GFA, SnapEDA Library:GCT_USB4110GFA, F.Cu at (33.2, 174.1)
- added R5: 5.1K, Resistor_SMD:R_1206_3216Metric_Pad1.30x1.75mm_HandSolder, F.Cu at (26.1, 165.2)
- added R7: 5.1K, Resistor_SMD:R_1206_3216Metric_Pad1.30x1.75mm_HandSolder, F.Cu at (30.6, 165.2)
- added U2: AMS1117-3.3, Package_TO_SOT_SMD:SOT-223-3_TabPin2, F.Cu at (60.6, 160.9)
- F1, F2: value Fuse -> 3522-2; footprint Fuse:Fuseholder_Clip-5x20mm_Eaton_1A5601-01_Inline_P20.80x6.76mm_D1.70mm_Horizontal -> fulse_holder_blade:FUSE_3522-2
- moved J1 14.4 mm to (18.9, 177.8)
- moved F2 10.2 mm to (17.3, 61.6)
- moved F1 9.16 mm to (18.6, 112.1)
- moved Y1 0.85 mm to (52.2, 148.1)
- moved J11 0.66 mm to (18.3, 84.0)
- moved J3 0.45 mm to (17.6, 44.5)
- moved J12 0.25 mm to (18.4, 132.5)
- moved C18 0.21 mm to (107.2, 83.2)
Connections:
- net Net-(D1-A) renamed +VDC
- C18 pad 1: +5V -> /junction1
- C21 pad 1: +5V -> /junction
- J5 pad 1: +5V -> +5C
- U3 pad 21: +3V3 -> unconnected-(U3-Pad21)
- U3 pad 22: +5V -> /junction
- U3 pad 27: +3V3 -> unconnected-(U3-Pad27)
- U5 pad 1: +5V -> VCC
- U6 pad 21: +3V3 -> unconnected-(U6-Pad21)
- U6 pad 22: +5V -> /junction1
- U6 pad 27: +3V3 -> unconnected-(U6-Pad27)
- U6 pad 28: +5V -> +5C
Routing:
- net +5V: track 322.6 -> 64.4 mm, vias 4 -> 1
- net +3V3: track 337.3 -> 100.3 mm, vias 6 -> 2
- net /junction: track 0.00 -> 186.7 mm, vias 0 -> 3
- net /junction1: track 0.00 -> 148.5 mm
- net VDD: track 0.00 -> 73.3 mm
- net VCC: track 151.1 -> 222.2 mm
- net +5C: track 0.00 -> 63.6 mm, vias 0 -> 1
- net unconnected-(U3-Pad21): track 0.00 -> 30.2 mm
- net /+: track 25.6 -> 52.1 mm
- net +VDC: track 29.1 -> 53.1 mm, vias 0 -> 3
- net /-: track 27.7 -> 47.4 mm
- net Net-(J7-CC1): track 0.00 -> 10.1 mm, vias 0 -> 2
- net Net-(J7-CC2): track 0.00 -> 9.57 mm, vias 0 -> 2
- net GND: track 3.13 -> 9.35 mm, vias 35 -> 40
- net RX1: track 148.5 -> 151.2 mm
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Other:
- board text added: "+"
- board text added: "-"
- board text added: "5V"
- board text added: "A"
- board text added: "A1"
- board text added: "B"
- board text added: "B1"
- board text added: "BOOT"
- board text added: "CAN_INTERFACE"
- board text added: "EXT_PWR"
- board text added: "G"
- board text added: "OD1_PWR"
- board text added: "OD2_PWR"
- board text added: "RESET"
- board text added: "RX"
- board text added: "TX"
- board text added: "UART"
- board text added: "VS"
- board text added: "Z"
- board text added: "Z1"

Commit message: updating finals ltst
Parts:
- added C19: 22UF, Capacitor_THT:CP_Radial_D8.0mm_P3.50mm, F.Cu at (40.3, 140.6)
- added H1: MountingHole, MountingHole:MountingHole_3.2mm_M3, F.Cu at (173.2, 19.3)
- added H2: MountingHole, MountingHole:MountingHole_3.2mm_M3, F.Cu at (173.6, 177.2)
- added H3: MountingHole, MountingHole:MountingHole_3.2mm_M3, F.Cu at (13.4, 165.4)
- added H4: MountingHole, MountingHole:MountingHole_3.2mm_M3, F.Cu at (30.2, 19.4)
- added J9: Conn_01x04_Pin, Connector_PinHeader_2.54mm:PinHeader_1x04_P2.54mm_Vertical, F.Cu at (168.8, 158.8)
- C1, C10, C11, C12, C2, C22, C3, C4, C5, C6, C7, C8, C9: value 100n -> 100nF
- moved C13 2.37 mm to (50.2, 143.2)
Routing:
- net H: track 125.4 -> 164.2 mm
- net VCC: track 222.2 -> 254.8 mm
- net L: track 112.6 -> 134.7 mm
- net Z12: track 45.1 -> 49.6 mm
- net B12: track 49.4 -> 53.4 mm
- net GND: track 9.35 -> 7.72 mm
- net Net-(U1-XI): track 21.6 -> 22.8 mm
Other:
- board text added: "CAN_H"
- board text added: "CAN_L"
- board text added: "GND"
- board text added: "VCC"

Commit message: addingg
Parts:
- removed J11: Screw_Terminal_01x02, TerminalBlock:TerminalBlock_Altech_AK300-2_P5.00mm
- added J13: B3B-PH-K-R_LF__SN_, SnapEDA Library:JST_B3B-PH-K-R_LF__SN_, F.Cu at (139.3, 144.2)
- added J14: B3B-PH-K-R_LF__SN_, SnapEDA Library:JST_B3B-PH-K-R_LF__SN_, F.Cu at (146.0, 144.1)
- added J15: B3B-PH-K-R_LF__SN_, SnapEDA Library:JST_B3B-PH-K-R_LF__SN_, F.Cu at (152.7, 144.2)
- added J16: B3B-PH-K-R_LF__SN_, SnapEDA Library:JST_B3B-PH-K-R_LF__SN_, F.Cu at (159.2, 144.2)
- added J17: B3B-PH-K-R_LF__SN_, SnapEDA Library:JST_B3B-PH-K-R_LF__SN_, F.Cu at (172.2, 144.2)
- added J18: B3B-PH-K-R_LF__SN_, SnapEDA Library:JST_B3B-PH-K-R_LF__SN_, F.Cu at (165.8, 144.2)
- added J19: Conn_01x02_Pin, Connector_AMASS:AMASS_XT30UPB-F_1x02_P5.0mm_Vertical, F.Cu at (20.7, 80.8)
- J4: footprint Connector_AMASS:AMASS_XT30UPB-M_1x02_P5.0mm_Vertical -> Connector_AMASS:AMASS_XT30UPB-F_1x02_P5.0mm_Vertical
- moved J4 3.33 mm to (20.8, 95.5)
Connections:
- F1 pad 1A: /fuse1 -> VDD
- F1 pad 1B: /fuse1 -> VDD
- F2 pad 2A: /onFuse -> /onFuse*
- F2 pad 2B: /onFuse -> /onFuse*
- J12 pad 2: /fuse1 -> VDD
- J4 pad 1: VDD -> GND
- U4 pad 11: unconnected-(U4-IO26-Pad11) -> /IO26
- U4 pad 12: unconnected-(U4-IO27-Pad12) -> /IO27
- U4 pad 13: unconnected-(U4-IO14-Pad13) -> /IO14
- U4 pad 14: unconnected-(U4-IO12-Pad14) -> /IO12
- U4 pad 16: unconnected-(U4-IO13-Pad16) -> /IO13
- U4 pad 9: unconnected-(U4-IO33-Pad9) -> /IO33
Routing:
- net /IO13: track 0.00 -> 90.7 mm, vias 0 -> 1
- net /IO12: track 0.00 -> 83.3 mm, vias 0 -> 1
- net /IO14: track 0.00 -> 75.6 mm, vias 0 -> 1
- net /IO27: track 0.00 -> 69.5 mm, vias 0 -> 1
- net /IO26: track 0.00 -> 62.3 mm, vias 0 -> 1
- net /IO33: track 0.00 -> 51.6 mm, vias 0 -> 1
- net VCC: track 254.8 -> 304.7 mm
- net VDD: track 73.2 -> 106.8 mm, vias 0 -> 12
- net L: track 134.7 -> 120.3 mm
- net /onFuse*: vias 0 -> 12
- net /onFuse: vias 0 -> 12
- net /fuse2: vias 0 -> 12
- added copper zone on B.Cu, net /fuse2
- added copper zone on B.Cu, net /onFuse
- added copper zone on B.Cu, net /onFuse*
- added copper zone on F.Cu, net /onFuse*
- added copper zone on B.Cu, net VDD
- removed copper zone on F.Cu, net /fuse1
Other:
- board text added: "VCC IO12 GND"
- board text added: "VCC IO13 GND"
- board text added: "VCC IO14 GND"
- board text added: "VCC IO26 GND"
- board text added: "VCC IO27 GND"
- board text added: "VCC IO33 GND"
