File: ODRIVE_V1.0.kicad_sch (KiCad schematic)
At the start: 48 parts, among them J1 USB_B, J10 RJ11-6N-B, J11 Screw_Terminal_01x02, J12 Screw_Terminal_01x02, J3 Screw_Terminal_01x02, J4 Conn_01x02_Pin, J5 Conn_01x08_Pin, J6 Conn_01x08_Pin, J8 Conn_01x04_Pin, SW3 SW_DPST_x2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

Commit message: updating to finals
Parts:
- removed C19, C20: 22UF, Capacitor_THT:CP_Radial_D8.0mm_P3.50mm, symbol Device:C_Polarized_Small_US
- removed F1, F2: Fuse, Fuse:Fuseholder_Clip-5x20mm_Eaton_1A5601-01_Inline_P20.80x6.76mm_D1.70mm_Horizontal, symbol Device:Fuse
- added C23, C24: 22UF, Capacitor_THT:CP_Radial_D5.0mm_P2.50mm, symbol Device:C_Polarized_Small_US
- added D2, D3: 1N4148, Diode_THT:D_DO-35_SOD27_P7.62mm_Horizontal, symbol Diode:1N4148
- added F1, F2: 3522-2, fulse_holder_blade:FUSE_3522-2, symbol fulse_holder_blade:3522-2
- added J2: Screw_Terminal_01x02, TerminalBlock:TerminalBlock_Altech_AK300-2_P5.00mm, symbol Connector:Screw_Terminal_01x02
- added J7: USB4110GFA, SnapEDA Library:GCT_USB4110GFA, symbol USB4110GFA:USB4110GFA
- added R5, R7: 5.1K, Resistor_SMD:R_1206_3216Metric_Pad1.30x1.75mm_HandSolder, symbol Device:R
- added U2: AMS1117-3.3, Package_TO_SOT_SMD:SOT-223-3_TabPin2, symbol Regulator_Linear:AMS1117-3.3
Connections:
- net +: now also J7.A6 (DP1), J7.B6 (DP2)
- net +3V3: now also C24.1, U2.2 (VO); no longer U3.21, U3.27, U6.21, U6.27
- net +5V: no longer C18.1, C21.1, J5.1 (Pin_1), U3.22, U5.1 (VCC), U6.22, U6.28
- net -: now also J7.A7 (DN1), J7.B7 (DN2)
- net GND: now also C23.2, C24.2, J2.2 (Pin_2), J7.A1/B12 (GND), J7.B1/A12 (GND__1), J7.S1 (GND__2), J7.S2 (GND__3), J7.S3 (GND__4), J7.S4 (GND__5), R5.2, R7.1, U2.1 (GND)
- net VCC: now also U5.1 (VCC), C23.1, D2.1 (K), D3.1 (K), U2.3 (VI)
- net VDD: now also J2.1 (Pin_1)
- net fuse1: now also F1.1A, F1.1B
- net fuse2: now also F2.1A, F2.1B
- net onFuse: now also F1.2A, F1.2B, F2.2A, F2.2B
- net +VDC: now reaches D1.2 (A), J1.1 (VBUS)
- net +VDC: now also J7.A4/B9 (VBUS), J7.B4/A9 (VBUS__1)
- new net: J7.A5 (CC1), R5.1
- new net: J7.B5 (CC2), R7.2
- new net +5C: J5.1 (Pin_1), U6.28
- new net junction: C21.1, D2.2 (A), U3.22
- new net junction1: C18.1, D3.2 (A), U6.22
- no-connect marks 63 -> 69
Other:
- moved on the sheet: C21, C22, J10, J12, R1, R2, U7

Commit message: updating finals ltst
Parts:
- added C19: 22UF, Capacitor_THT:CP_Radial_D8.0mm_P3.50mm, symbol Device:C_Polarized_Small_US
- added H1, H2, H3, H4: MountingHole, MountingHole:MountingHole_3.2mm_M3, symbol Mechanical:MountingHole
- added J9: Conn_01x04_Pin, Connector_PinHeader_2.54mm:PinHeader_1x04_P2.54mm_Vertical, symbol Connector:Conn_01x04_Pin
- C1, C10, C11, C12, C2, C22, C3, C4, C5, C6, C7, C8, C9: value 100n -> 100nF
Connections:
- net GND: now also C19.2, J9.4 (Pin_4)
- net H: now also J9.2 (Pin_2)
- net L: now also J9.3 (Pin_3)
- net VCC: now also C19.1, J9.1 (Pin_1)

Commit message: addingg
Parts:
- removed J11: Screw_Terminal_01x02, TerminalBlock:TerminalBlock_Altech_AK300-2_P5.00mm, symbol Connector:Screw_Terminal_01x02
- added J13, J14, J15, J16, J17, J18: B3B-PH-K-R_LF__SN_, SnapEDA Library:JST_B3B-PH-K-R_LF__SN_, symbol B3B-PH-K-R_LF__SN_:B3B-PH-K-R_LF__SN_
- added J19: Conn_01x02_Pin, Connector_AMASS:AMASS_XT30UPB-F_1x02_P5.0mm_Vertical, symbol Connector:Conn_01x02_Pin
- J4: footprint Connector_AMASS:AMASS_XT30UPB-M_1x02_P5.0mm_Vertical -> Connector_AMASS:AMASS_XT30UPB-F_1x02_P5.0mm_Vertical
Connections:
- net fuse1 is gone; now on net VDD: F1.1A, F1.1B, J12.2 (Pin_2)
- net GND: now also J4.1 (Pin_1), J13.3, J14.3, J15.3, J16.3, J17.3, J18.3, J19.1 (Pin_1)
- net VCC: now also J13.1, J14.1, J15.1, J16.1, J17.1, J18.1
- net VDD: no longer J4.1 (Pin_1)
- net onFuse: no longer F2.2A, F2.2B
- net IO26: now reaches U4.11 (IO26)
- net IO26: now also J14.2
- net IO27: now reaches U4.12 (IO27)
- net IO27: now also J15.2
- net IO14: now reaches U4.13 (IO14)
- net IO14: now also J16.2
- net IO12: now reaches U4.14 (IO12)
- net IO12: now also J18.2
- net IO13: now reaches U4.16 (IO13)
- net IO13: now also J17.2
- net IO33: now reaches U4.9 (IO33)
- net IO33: now also J13.2
- new net onFuse*: F2.2A, F2.2B, J19.2 (Pin_2)
- no-connect marks 69 -> 63
Other:
- moved on the sheet: F1, J12
